File: TSOC_GROVEY_GPIO/revisions/R2_0/TSOC_GROVEY_GPIO.brd (EAGLE design)
At the start: 44.5 x 30.5 mm, 60 parts, among them J1 4P-2.0-90D, J2 4P-2.0-90D, J3 4P-2.0-90D, J4 4P-2.0-90D, Q1 CJ2305, Q2 CJ2305, Q3 BSS138W-7-F, Q4 BSS138W-7-F, Q5 BSS138W-7-F, Q6 BSS138W-7-F, Q7 CJ2305, Q8 CJ2305, U1 SX1509

Commit message: update to Rev2.0
Parts:
- removed A0: NO, scratch-ProtoPads:JMP-2-NO
- added A2: NO, scratch-ProtoPads:JMP-2-NO
- added R15, R16: 47K, Seeed-Resistor-2016:R0603
- added R17, R18: 1K 1/10W, Seeed-Resistor-2016:R0603
- C3: value 100uf -> 10uf
- C8: value 1uf -> 10uf; device Seeed-Capacitor-2016:C0603 -> Seeed-Capacitor-2016:C1206
- C9: value 100uf -> 1uf; device Seeed-Capacitor-2016:C1206 -> Seeed-Capacitor-2016:C0603
- R11: value 47K -> 10K 1/10W
- R13: value 1K 1/10W -> 47K
- R14: value 1K 1/10W -> 10K 1/10W
- R5, R6: value 10K 1/10W -> 47K
- moved R7 19.0 mm to (15.2, 6.35)
- moved R10 17.5 mm to (24.4, 6.86)
- moved A1 17.2 mm to (22.6, 6.86), turned to 0 degrees
- moved R9 17.0 mm to (23.1, 23.6)
- moved R13 15.6 mm to (26.7, 11.2), turned to 180 degrees
- moved R5 11.5 mm to (14.5, 18.0), turned to 90 degrees
- moved R14 11.2 mm to (29.5, 23.6), turned to 180 degrees
- moved R4 10.1 mm to (11.7, 8.64), turned to 270 degrees
- moved R3 9.68 mm to (11.2, 18.0)
- moved C8 7.71 mm to (31.2, 14.0), turned to 0 degrees
- moved C9 7.71 mm to (33.5, 6.60), turned to 90 degrees
- moved R11 7.58 mm to (25.9, 6.86), turned to 180 degrees
- moved R8 7.38 mm to (17.0, 6.35)
- moved R12 6.43 mm to (26.2, 20.1), turned to 270 degrees
- moved R6 3.06 mm to (14.7, 8.64), turned to 90 degrees
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- renumbered $$U$4 to $$U$1, $$U$5 to $$U$2
Connections:
- net !INT: now also R14.1; no longer R10.1
- net !RST: now also R11.1; no longer R9.1
- net 3V3: now also R11.2, R14.2; no longer R5.2, R6.2
- net A0: now also A1.2, R10.1; no longer A0.2, R8.1
- net A1: now also A2.2, R9.1; no longer A1.2, R7.1
- net GND: now also A2.1, Q3.2, Q4.2, Q5.2, Q6.2, R12.1, R13.1, R5.1, R6.1; no longer A0.1, Q3.3, Q4.3, Q5.3, Q6.3
- net IO10: now also R5.2
- net IO14: now also R6.2
- net IO2: now also R13.2
- net IO3: now also R17.2; no longer R13.2
- net IO6: now also R12.2
- net IO7: now also R18.2; no longer R14.2
- net LED2: now also R18.1; no longer R14.1
- net LED3: now also R17.1; no longer R13.1
- net N$1: now also Q4.3, R3.1; no longer Q4.2, R4.1
- net N$2: now also Q3.3, R4.1; no longer Q3.2, R3.1
- net N$3: now also Q5.3, R15.1; no longer Q5.2, R11.1
- net N$4: now also Q6.3, R16.1; no longer Q6.2, R12.1
- net SCL: now also R8.1; no longer R6.1
- net SDA: now also R7.1; no longer R5.1
- net VCC: now also C8.2, R15.2, R16.2; no longer C9.2, R11.2, R12.2
- net VCC1: now also C9.2; no longer C8.2
Routing:
- net GND: track 263.5 -> 271.5 mm, vias 16 -> 17
- net IO2: track 11.2 -> 7.54 mm
- net VCC: track 92.0 -> 95.2 mm
- net IO14: track 12.8 -> 10.5 mm
- net IO10: track 13.1 -> 14.9 mm
- net N$3: track 3.18 -> 4.12 mm
- net N$4: track 3.18 -> 4.09 mm
- net N$1: track 3.17 -> 4.05 mm
- net !RST: track 18.7 -> 17.9 mm
- net IO5: track 17.6 -> 18.1 mm
- net IO6: track 8.18 -> 7.83 mm, vias 2 -> 0
Other:
- board text added: "Rev. 2.0"
- board text removed: "Rev. 1.1"
