File: TSOC_GROVEY_GPIO/revisions/R2_0/TSOC_GROVEY_GPIO.sch (EAGLE design)
At the start: 57 parts, among them J1 4P-2.0-90D, J2 4P-2.0-90D, J3 4P-2.0-90D, J4 4P-2.0-90D, Q1 CJ2305, Q2 CJ2305, Q3 BSS138W-7-F, Q4 BSS138W-7-F, Q5 BSS138W-7-F, Q6 BSS138W-7-F, Q7 CJ2305, Q8 CJ2305, U1 SX1509

Commit message: update to Rev2.0
Parts:
- removed A0: NO, scratch-ProtoPads:JMP-2-NO
- added A2: NO, scratch-ProtoPads:JMP-2-NO
- added R15, R16: 47K, Seeed-Resistor-2016:SMD-RES-47K-5%-1/10W(0603)
- added R17, R18: 1K 1/10W, Seeed-Resistor-2016:SMD-RES-1K-5%-1/10W(0603)
- C3: value 100uf -> 10uf; device Seeed-Capacitor-2016:CERAMIC-100UF-6.3V-20%-X5R(1206) -> Seeed-Capacitor-2016:CERAMIC-10UF-25V-10%-X5R(1206)
- C8: value 1uf -> 10uf; device Seeed-Capacitor-2016:CERAMIC-1UF-25V-10%-X7R(0603) -> Seeed-Capacitor-2016:CERAMIC-10UF-25V-10%-X5R(1206)
- C9: value 100uf -> 1uf; device Seeed-Capacitor-2016:CERAMIC-100UF-6.3V-20%-X5R(1206) -> Seeed-Capacitor-2016:CERAMIC-1UF-25V-10%-X7R(0603)
- R11: value 47K -> 10K 1/10W; device Seeed-Resistor-2016:SMD-RES-47K-5%-1/10W(0603) -> Seeed-Resistor-2016:SMD-RES-10K-5%-1/10W(0603)
- R13: value 1K 1/10W -> 47K; device Seeed-Resistor-2016:SMD-RES-1K-5%-1/10W(0603) -> Seeed-Resistor-2016:SMD-RES-47K-5%-1/10W(0603)
- R14: value 1K 1/10W -> 10K 1/10W; device Seeed-Resistor-2016:SMD-RES-1K-5%-1/10W(0603) -> Seeed-Resistor-2016:SMD-RES-10K-5%-1/10W(0603)
- R5, R6: value 10K 1/10W -> 47K; device Seeed-Resistor-2016:SMD-RES-10K-5%-1/10W(0603) -> Seeed-Resistor-2016:SMD-RES-47K-5%-1/10W(0603)
- renumbered $$U$4 to $$U$1, $$U$5 to $$U$2
Connections:
- net !INT: now also R14.1; no longer R10.1
- net !RST: now also R11.1; no longer R9.1
- net 3V3: now also R11.2, R14.2; no longer R5.2, R6.2
- net A0: now also A1.2, R10.1; no longer A0.2, R8.1
- net A1: now also A2.2, R9.1; no longer A1.2, R7.1
- net GND: now also A2.1, Q3.S, Q4.S, Q5.S, Q6.S, R12.1, R13.1, R5.1, R6.1; no longer A0.1, Q3.D, Q4.D, Q5.D, Q6.D
- net IO10: now also R5.2
- net IO14: now also R6.2
- net IO2: now also R13.2
- net IO3: now also R17.2; no longer R13.2
- net IO6: now also R12.2
- net IO7: now also R18.2; no longer R14.2
- net LED2: now also R18.1; no longer R14.1
- net LED3: now also R17.1; no longer R13.1
- net N$1: now also Q4.D, R3.1; no longer Q4.S, R4.1
- net N$2: now also Q3.D, R4.1; no longer Q3.S, R3.1
- net N$3: now also Q5.D, R15.1; no longer Q5.S, R11.1
- net N$4: now also Q6.D, R16.1; no longer Q6.S, R12.1
- net SCL: now also R8.1; no longer R6.1
- net SDA: now also R7.1; no longer R5.1
- net VCC: now also C8.2, R15.2, R16.2; no longer C9.2, R11.2, R12.2
- net VCC1: now also C9.2; no longer C8.2
Other:
- moved on the sheet: A1, C8, C9, Q3, Q4, Q5, Q6, R10, R11, R12, R13, R14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
